File: Arduino-Media-Player.sch (EAGLE design)
At the start: 41 parts, among them IC1 AMS117-18, IC2 AMS117-33, U1 VS1053B, U2 FT232RLSSOP, U3 ATMEGA328P, U4 DS1307SO8, U5 74HC4050 LVL CONVERTER

Commit message: Few minor changes
Parts:
- removed FRAME1: FRAME-LETTER, SparkFun-Aesthetics:FRAME-LETTER
